Commit message: add ultrasonic to urdf

File: src/description/marvin_description/urdf/constants.xacro (robot description, xacro)
@@ -43,3 +43,7 @@
     <xacro:property name="gps_y_offset" value="0.0"/>
     <xacro:property name="gps_z_offset" value="${chassis_z_offset + chassis_tower_height}"/>
+    <!-- Rear Ultrasonic Sensor Constants -->
+    <xacro:property name="ultrasonic_rear_x_offset" value="${-(chassis_tower_length/2 + chassis_electrical_length + chassis_caster_length)}"/>
+    <xacro:property name="ultrasonic_rear_y_spacing" value="${8*0.0254}"/>
+    <xacro:property name="ultrasonic_rear_z_offset" value="${chassis_z_offset + 2*0.0254}"/>
 </robot>

File: src/description/marvin_description/urdf/marvin.xacro (robot description, xacro)
@@ -40,3 +40,14 @@
         <origin xyz="${gps_x_offset} ${gps_y_offset} ${gps_z_offset}" rpy="0 0 0" />
     </xacro:ann_mb>
+    <!-- Rear Ultrasonic Sensors -->
+    <xacro:include filename="$(find common_description)/urdf/sensor/ultrasonic.xacro" />
+    <xacro:ultrasonic name="ultrasonic_rear_left" parent="$(arg base_frame_id)">
+        <origin xyz="${ultrasonic_rear_x_offset} ${ultrasonic_rear_y_spacing} ${ultrasonic_rear_z_offset}" rpy="0 0 ${pi}" />
+    </xacro:ultrasonic>
+    <xacro:ultrasonic name="ultrasonic_rear_center" parent="$(arg base_frame_id)">
+        <origin xyz="${ultrasonic_rear_x_offset} 0 ${ultrasonic_rear_z_offset}" rpy="0 0 ${pi}" />
+    </xacro:ultrasonic>
+    <xacro:ultrasonic name="ultrasonic_rear_right" parent="$(arg base_frame_id)">
+        <origin xyz="${ultrasonic_rear_x_offset} ${-ultrasonic_rear_y_spacing} ${ultrasonic_rear_z_offset}" rpy="0 0 ${pi}" />
+    </xacro:ultrasonic>
 </robot>
